File: PCB/A4960 Devboard.kicad_pcb (KiCad board)
At the start: 2 copper layers, 43.4 x 48.8 mm, 58 parts, among them IC1 ATMEGA8-AI, P1 CONN_02X03, P2 CONN_01X02, P3 CONN_01X03, P4 CONN_01X03, Q1 Q_NMOS_GDS_old, Q2 Q_NMOS_GDS_old, Q3 Q_NMOS_GDS_old, Q4 Q_NMOS_GDS_old, Q5 Q_NMOS_GDS_old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

Commit message: PowerPole-Stecker korrigiert
Routing:
- net Net-(C15-Pad2): track 6.92 -> 8.50 mm
Changed lines of the file:
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@@
     (thickness 1.6)
     (drawings 72)
-    (tracks 863)
+    (tracks 864)
     (zones 0)
     (modules 58)
@@
   (layers
     (0 F.Cu signal)
-    (31 B.Cu signal hide)
+    (31 B.Cu signal)
     (32 B.Adhes user)
     (33 F.Adhes user)
@@
     (add_net VPP)
   )
+  (module Pin_Headers:Pin_Header_Straight_1x02 (layer F.Cu)
+    (at 197.231 69.596)
+    (descr "Through hole pin header")
+    (tags "pin header")
+    (fp_text reference P2 (at 0 -5.1) (layer F.SilkS)
+      (effects (font (size 1 1) (thickness 0.15)))
+    )
+    (fp_text value CONN_01X02 (at 0 -3.1) (layer F.Fab)
+      (effects (font (size 1 1) (thickness 0.15)))
+    )
+    (pad 1 thru_hole oval (at 0 0) (size 3 5) (drill oval 2 4.5) (layers *.Cu *.Mask F.SilkS)
+      (net 7 VPP) (zone_connect 2))
+    (pad 2 thru_hole oval (at 0 7.9) (size 3 5) (drill oval 2 4.5) (layers *.Cu *.Mask F.SilkS)
+      (net 2 GND) (zone_connect 2))
+    (model Pin_Headers.3dshapes/Pin_Header_Straight_1x02.wrl
+      (at (xyz 0 -0.05 0))
+      (scale (xyz 1 1 1))
+      (rotate (xyz 0 0 90))
+    )
+  )
   (module Pin_Headers:Pin_Header_Straight_1x03 (layer F.Cu)
     (at 213.995 76.073 90)
@@
       (effects (font (size 1 1) (thickness 0.15)))
     )
-    (pad 1 thru_hole oval (at 0 0 90) (size 3 5) (drill oval 2 4) (layers *.Cu *.Mask F.SilkS)
+    (pad 1 thru_hole oval (at 0 0 90) (size 3 5) (drill oval 2 4.5) (layers *.Cu *.Mask F.SilkS)
       (net 13 /MotorA) (zone_connect 2))
-    (pad 2 thru_hole oval (at 0 7.9 90) (size 3 5) (drill oval 2 4) (layers *.Cu *.Mask F.SilkS)
+    (pad 2 thru_hole oval (at 0 7.9 90) (size 3 5) (drill oval 2 4.5) (layers *.Cu *.Mask F.SilkS)
       (net 15 /MotorB) (zone_connect 2))
-    (pad 3 thru_hole oval (at 0 15.8 90) (size 3 5) (drill oval 2 4) (layers *.Cu *.Mask F.SilkS)
+    (pad 3 thru_hole oval (at 0 15.8 90) (size 3 5) (drill oval 2 4.5) (layers *.Cu *.Mask F.SilkS)
       (net 17 /MotorC) (zone_connect 2))
     (model Pin_Headers.3dshapes/Pin_Header_Straight_1x03.wrl
@@
       (scale (xyz 1 1 1))
       (rotate (xyz 0 0 0))
-    )
-  )
-  (module Pin_Headers:Pin_Header_Straight_1x02 (layer F.Cu)
-    (at 197.231 69.596)
-    (descr "Through hole pin header")
-    (tags "pin header")
-    (fp_text reference P2 (at 0 -5.1) (layer F.SilkS)
-      (effects (font (size 1 1) (thickness 0.15)))
-    )
-    (fp_text value CONN_01X02 (at 0 -3.1) (layer F.Fab)
-      (effects (font (size 1 1) (thickness 0.15)))
-    )
-    (fp_line (start 1.27 1.27) (end 1.27 3.81) (layer F.SilkS) (width 0.15))
-    (fp_line (start 1.55 -1.55) (end 1.55 0) (layer F.SilkS) (width 0.15))
-    (fp_line (start -1.75 -1.75) (end -1.75 4.3) (layer F.CrtYd) (width 0.05))
-    (fp_line (start 1.75 -1.75) (end 1.75 4.3) (layer F.CrtYd) (width 0.05))
-    (fp_line (start -1.75 -1.75) (end 1.75 -1.75) (layer F.CrtYd) (width 0.05))
-    (fp_line (start -1.75 4.3) (end 1.75 4.3) (layer F.CrtYd) (width 0.05))
-    (fp_line (start 1.27 1.27) (end -1.27 1.27) (layer F.SilkS) (width 0.15))
-    (fp_line (start -1.55 0) (end -1.55 -1.55) (layer F.SilkS) (width 0.15))
-    (fp_line (start -1.55 -1.55) (end 1.55 -1.55) (layer F.SilkS) (width 0.15))
-    (fp_line (start -1.27 1.27) (end -1.27 3.81) (layer F.SilkS) (width 0.15))
-    (fp_line (start -1.27 3.81) (end 1.27 3.81) (layer F.SilkS) (width 0.15))
-    (pad 1 thru_hole oval (at 0 0) (size 3 5) (drill oval 2 4) (layers *.Cu *.Mask F.SilkS)
-      (net 7 VPP) (zone_connect 2))
-    (pad 2 thru_hole oval (at 0 7.9) (size 3 5) (drill oval 2 4) (layers *.Cu *.Mask F.SilkS)
-      (net 2 GND) (zone_connect 2))
-    (model Pin_Headers.3dshapes/Pin_Header_Straight_1x02.wrl
-      (at (xyz 0 -0.05 0))
-      (scale (xyz 1 1 1))
-      (rotate (xyz 0 0 90))
     )
   )
@@
   (segment (start 223.913 102.858) (end 223.913 103.505) (width 0.508) (layer F.Cu) (net 10))
   (segment (start 224.136 102.635) (end 223.913 102.858) (width 0.508) (layer F.Cu) (net 10))
+  (segment (start 223.024 107.188) (end 223.024 108.7628) (width 0.254) (layer F.Cu) (net 11))
   (segment (start 223.163 105.283) (end 223.163 107.049) (width 0.254) (layer F.Cu) (net 11))
   (segment (start 223.163 107.049) (end 223.024 107.188) (width 0.254) (layer F.Cu) (net 11))

Commit message: Credits angegeben
Other:
- board text added: "(C) Sven T. Schneider"
- board text removed: "Sven Schneider"
Changed lines of the file:
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@@
-(kicad_pcb (version 4) (host pcbnew 0.201511171411+6319~30~ubuntu15.10.1-product)
+(kicad_pcb (version 4) (host pcbnew 0.201512031508+6343~38~ubuntu15.10.1-stable)
   (general
     (links 256)
@@
   (gr_line (start 219 102.5) (end 218.5 102) (angle 90) (layer B.Mask) (width 0.5))
   (gr_line (start 224.5 97) (end 219 102.5) (angle 90) (layer B.Mask) (width 0.5))
-  (gr_text "Sven Schneider\n" (at 194.5 92 270) (layer B.SilkS)
-    (effects (font (size 1.5 1.5) (thickness 0.3)) (justify mirror))
-  )
-  (gr_text "(C) Philipp Hörauf\n" (at 197 94.5 270) (layer B.SilkS)
-    (effects (font (size 1.5 1.5) (thickness 0.3)) (justify mirror))
+  (gr_text "(C) Sven T. Schneider\n" (at 193.421 98.933 270) (layer F.SilkS)
+    (effects (font (size 1 1) (thickness 0.15)))
+  )
+  (gr_text "(C) Philipp Hörauf\n" (at 193.421 75.692 270) (layer F.SilkS)
+    (effects (font (size 1 1) (thickness 0.15)))
   )
   (gr_line (start 227.5 69) (end 228 69) (angle 90) (layer B.Mask) (width 0.5))

Commit message: Leiterplatte so gefertigt
Parts:
- R10: value R -> 5,6k
- R3: value R -> 22k
- R4: value R -> 2,2k
- R5, R8: value 100 -> 330
- R9: value R -> 10k
Connections:
- P1 pad 1: /MOSI -> /MISO
- P1 pad 4: /MISO -> /MOSI
Routing:
- net /SCK: track 15.8 -> 19.0 mm
- net /MOSI: track 17.7 -> 19.7 mm
- net /MISO: track 14.4 -> 16.3 mm

Commit message: last commit des "alten" Standes von 2016
Other:
- net class Default removed
