File: PCB/A4960 Devboard.sch (KiCad schematic (older format))
At the start: 60 parts, among them IC1 ATMEGA8-AI, P1 CONN_02X03, P2 CONN_01X02, P3 CONN_01X03, P4 CONN_01X03, P5 CONN_01X03, P6 CONN_01X03, Q1 SIRA00DP-T1-GE3, Q2 SIRA00DP-T1-GE3, Q3 SIRA00DP-T1-GE3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

Commit message: last commit des "alten" Standes von 2016
Parts:
- C1, C10, C11, C12, C13, C14, C15, C16, C17, C18, C19, C2, C20, C23, C3, C4, C8, C9: symbol C -> A4960-Devboard-rescue:C
- C21: symbol CP -> A4960-Devboard-rescue:CP
- D1: symbol ZENER -> A4960-Devboard-rescue:ZENER
- D3, D4: symbol LED -> A4960-Devboard-rescue:LED
- IC1: symbol ATMEGA8-AI -> A4960-Devboard-rescue:ATMEGA8-AI
- P1: symbol CONN_02X03 -> A4960-Devboard-rescue:CONN_02X03
- P2: symbol CONN_01X02 -> A4960-Devboard-rescue:CONN_01X02
- P3, P4, P5, P6: symbol CONN_01X03 -> A4960-Devboard-rescue:CONN_01X03
- Q1, Q2, Q3, Q4, Q5, Q6: symbol Q_NMOS_GDS_old -> A4960-Devboard-rescue:Q_NMOS_GDS_old
- R1, R10, R11, R12, R13, R14, R15, R16, R17, R18, R19, R2, R20, R21, R3, R4, R5, R6, R7, R8, R9: symbol R -> A4960-Devboard-rescue:R
- RP1: symbol R_PACK4 -> A4960-Devboard-rescue:R_PACK4
- U1: symbol AP1117D50 -> A4960-Devboard-rescue:AP1117D50
- U2: symbol A4960 -> ph-motor:A4960
- Y1: symbol RESONATEUR -> Resonator_3pins:RESONATEUR
